File: power.kicad_sch (KiCad schematic)
At the start: 6 parts, among them J7 Conn_01x02, U1 RK3562, U3 RT9992ZQW

Commit message: i understand
Parts:
- added C29, C30, C31, C32: 10uF, symbol Device:C
- added C33: 0.1uF, Capacitor_SMD:C_0402_1005Metric, symbol Device:C
- added D1: D, symbol Device:D
- added J9: Conn_01x02, Connector_JST:JST_PH_S2B-PH-K_1x02_P2.00mm_Horizontal, symbol Connector_Generic:Conn_01x02
- added L2: 2.2uH, footprints:IND-SMD_L5.8-W5.2_SLF05XX, symbol Device:L
- added L3: 8.2uH, footprints:IND-SMD_L5.8-W5.2_SLF05XX, symbol Device:L
- added R10, R11, R8: 20K, PCM_Resistor_SMD_AKL:R_0402_1005Metric, symbol Device:R
- added R9: 160K, PCM_Resistor_SMD_AKL:R_0402_1005Metric, symbol Device:R
- added SW1: SW_DP3T, symbol Switch:SW_DP3T
- added U5: TPS54360DDA, Package_SO:TI_SO-PowerPAD-8_ThermalVias, symbol Regulator_Switching:TPS54360DDA
- R6: value 20k -> 470k
- R7: value 160k -> 88.7k
Connections:
- net +BATT: now also U3.21 (PVDD3), C29.1, C30.1, C31.1, C32.1, SW1.3; no longer J7.1 (Pin_1)
- net GNDPWR: now also C29.2, C30.2, C31.2, C32.2, D1.2 (A), R11.2, R9.2, SW1.7, U5.7 (GND), U5.9 (GNDPAD)
- net +5V: now reaches R6.1, U3.30 (PVDD1)
- net at U3.18 (FB3): now also R8.2, R9.1
- net at U3.20 (LX3): now also L2.1
- new net: L2.2, R8.1
- new net: C33.1, U5.1 (BOOT)
- new net: C33.2, L3.2, R10.1, SW1.1
- new net: J7.1 (Pin_1), U5.2 (VIN)
- new net: R10.2, R11.1, U5.5 (FB)
- new net: D1.1 (K), L3.1, U5.8 (SW)
- new net: J9.1 (Pin_1), SW1.4
Other:
- moved on the sheet: J7
